Commit message: Update finalized version

File: mycobot_description/urdf/myarm_m750/myarm_m750_poe_v3_1.urdf (robot description, URDF)
Before this commit: robot myarm_m750, 11 links, 10 joints
Joints:
- joint left_gripper_joint: type prismatic -> fixed
- joint right_gripper_joint: type prismatic -> fixed
